File: pcb/tomato_timer.kicad_pcb (KiCad board)
At the start: 2 copper layers, 68.6 x 53.3 mm, 28 parts, among them J1 External_Power, Q1 BSS138, Q2 BSS138, Q3 TRANSISTOR_NPN, SW2 SW_Reset, SW3 SW_Start, SW4 SW_Stop, U1 XBeeSeries1

Commit message: Final board build used for fabrication.
Parts:
- removed JP1: Jumper_2_Open, Pin_Headers:Pin_Header_Straight_1x02_Pitch2.54mm
- D1: footprint tomato-timer:SSW-104-02-G-S-RA_4POS_Female_Header -> Connectors_JST:JST_PH_S3B-PH-K_03x2.00mm_Angled
- moved C1 6.13 mm to (176.4, 95.0), turned to 180 degrees
- moved R8 5.12 mm to (194.3, 68.5)
- moved R7 4.53 mm to (199.3, 75.2), turned to 180 degrees
- moved R5 4.03 mm to (203.9, 70.5), turned to 270 degrees
- moved JP2 3.21 mm to (165.5, 68.8), turned to 0 degrees
- moved R4 1.68 mm to (174.0, 100.4)
- moved D1 1.58 mm to (188.9, 68.5), turned to 180 degrees
- moved C3 1.37 mm to (187.4, 106.8), turned to 270 degrees
- moved C2 1.35 mm to (157.3, 78.7)
- moved R9 0.96 mm to (202.0, 104.7), turned to 180 degrees
- moved J1 0.79 mm to (158.9, 66.0)
- moved R3 0.70 mm to (165.2, 83.7)
Connections:
- C2 pad 2: /GND_IN -> /GND
- D1 pad 1: (no net) -> Net-(D1-Pad1)
- D1 pad 2: /GND_IN -> /5V_IN
- D1 pad 3: /5V_IN -> /GND
- D2 pad 2: /GND_IN -> /GND
- J1 pad 2: /GND_IN -> /GND
- LS1 pad 2: Net-(LS1-Pad2) -> /VOL_IN
- R10 pad 1: Net-(LS1-Pad2) -> /VOL_IN
- R8 pad 1: Net-(D1-Pad4) -> Net-(D1-Pad1)
- RV1 pad 2: Net-(LS1-Pad2) -> /VOL_IN
- TOMATO_SHIELD1 pad 7: (no net) -> /PIXEL_STRIP_PIN
- TOMATO_SHIELD1 pad 8: /PIXEL_STRIP_PIN -> (no net)
- TOMATO_SHIELD1 pad AD0: /BUZZER -> (no net)
- TOMATO_SHIELD1 pad AD1: (no net) -> /BUZZER
- TOMATO_SHIELD1 pad AD4: (no net) -> /VOL_IN
Routing:
- net /GND_IN: track 109.5 -> 0.00 mm
- net /VOL_IN: track 0.00 -> 88.8 mm
- net Net-(LS1-Pad2): track 37.9 -> 0.00 mm
- net /5V_IN: track 74.4 -> 38.4 mm
- net /GND: track 3.10 -> 15.2 mm
- net Net-(D1-Pad4): track 8.10 -> 0.00 mm
- net /PIXEL_STRIP_PIN: track 10.1 -> 3.00 mm
- net Net-(D1-Pad1): track 0.00 -> 7.04 mm
- net /TX: track 68.1 -> 62.4 mm, vias 4 -> 2
- net Net-(D2-Pad4): track 3.77 -> 8.58 mm
- net /5V: track 152.3 -> 148.0 mm, vias 3 -> 0
- net Net-(Q3-PadB): track 3.76 -> 7.91 mm
- net /RX: track 74.6 -> 70.5 mm
- net /PIXEL_RING_PIN: track 15.5 -> 12.4 mm
- net /BTN_START: track 84.4 -> 86.2 mm
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- added copper zone on F.Cu, net /5V_IN
Other:
- rule trace_min: 0.2 -> 0.15
- board text added: "DO"
- board text removed: "IN"
- board text removed: "OUT"
